Commit message: working prob arm controlled on my platform

File: nsc_robot_description/urdf/nsc_robot_with_p_rob.xacro (robot description, xacro)
@@ -1,7 +1,7 @@
 <?xml version="1.0"?>
 <robot name="nsc_robot" xmlns:xacro="http://www.ros.org/wiki/xacro">
- <xacro:include filename="$(find nsc_robot_description)/urdf/nsc_robot_arm.xacro" />
+ <xacro:include filename="$(find nsc_robot_p_arm_description)/urdf/p_arm.urdf.xacro" />
  <xacro:include filename="$(find nsc_robot_description)/urdf/nsc_robot_platform.xacro" />
- <xacro:include filename="$(find nsc_robot_description)/urdf/nsc_robot.gazebo" />
+ <xacro:include filename="$(find nsc_robot_description)/urdf/nsc_robot_with_prob.gazebo" />
  <!-- Constants for robot dimensions -->
   <xacro:property name="PI" value="3.1415926535897931"/>
@@ -17,7 +17,11 @@
   <xacro:property name="camera_link" value="0.05" />
   <xacro:property name="axel_offset" value="0.05" />
+    <xacro:property name="joint1_frame_rotation" value="0.0" />
+  <xacro:p_arm name="lio" parent="base_link" version="p_rob_2R">
+    <origin xyz="0 0 0.212" rpy="0 0 ${joint1_frame_rotation}" />
+  </xacro:p_arm>
   <transmission name="tran1">
     <type>transmission_interface/SimpleTransmission</type>
-    <joint name="joint_arm1">
+    <joint name="lio_joint1">
       <hardwareInterface>EffortJointInterface</hardwareInterface>
     </joint>
@@ -29,5 +33,5 @@
   <transmission name="tran2">
     <type>transmission_interface/SimpleTransmission</type>
-    <joint name="joint_arm2">
+    <joint name="lio_joint2">
       <hardwareInterface>EffortJointInterface</hardwareInterface>
     </joint>
@@ -39,5 +43,5 @@
   <transmission name="tran3">
     <type>transmission_interface/SimpleTransmission</type>
-    <joint name="joint_arm3">
+    <joint name="lio_joint3">
       <hardwareInterface>EffortJointInterface</hardwareInterface>
     </joint>
@@ -47,3 +51,33 @@
     </actuator>
   </transmission>
+    <transmission name="tran4">
+    <type>transmission_interface/SimpleTransmission</type>
+    <joint name="lio_joint4">
+      <hardwareInterface>EffortJointInterface</hardwareInterface>
+    </joint>
+    <actuator name="motor4">
+      <hardwareInterface>EffortJointInterface</hardwareInterface>
+      <mechanicalReduction>1</mechanicalReduction>
+    </actuator>
+  </transmission>
+  <transmission name="tran5">
+    <type>transmission_interface/SimpleTransmission</type>
+    <joint name="lio_joint5">
+      <hardwareInterface>EffortJointInterface</hardwareInterface>
+    </joint>
+    <actuator name="motor5">
+      <hardwareInterface>EffortJointInterface</hardwareInterface>
+      <mechanicalReduction>1</mechanicalReduction>
+    </actuator>
+  </transmission>
+    <transmission name="tran6">
+    <type>transmission_interface/SimpleTransmission</type>
+    <joint name="lio_joint6">
+      <hardwareInterface>EffortJointInterface</hardwareInterface>
+    </joint>
+    <actuator name="motor6">
+      <hardwareInterface>EffortJointInterface</hardwareInterface>
+      <mechanicalReduction>1</mechanicalReduction>
+    </actuator>
+  </transmission>
 </robot>

Commit message: added wheels - working lio with gripper and platform

File: nsc_robot_description/urdf/nsc_robot_with_p_rob.xacro (robot description, xacro)
@@ -1,8 +1,12 @@
 <?xml version="1.0"?>
 <robot name="nsc_robot" xmlns:xacro="http://www.ros.org/wiki/xacro">
+ <xacro:property name="robot_type" value="$(env ROBOT_TYPE)"/>
+ <xacro:property name="robot_base_frame_rotation" value="$(env RDSCFG_fp_descriptions_robot_frame_rotation)"/>
+ <xacro:property name="joint1_frame_rotation" value="$(env RDSCFG_fp_descriptions_j1_frame_rotation)"/>
  <xacro:include filename="$(find nsc_robot_p_arm_description)/urdf/p_arm.urdf.xacro" />
- <xacro:include filename="$(find nsc_robot_description)/urdf/nsc_robot_platform.xacro" />
+ <!-- <xacro:include filename="$(find nsc_robot_description)/urdf/nsc_robot_platform.xacro" /> -->
  <xacro:include filename="$(find nsc_robot_description)/urdf/nsc_robot_with_prob.gazebo" />
  <xacro:include filename="$(find nsc_robot_p_grip_description)/urdf/p_grip.urdf.xacro" />
+ <xacro:include filename="$(find nsc_robot_platform_description)/urdf/platform_${robot_type}.urdf.xacro" />
  <!-- Constants for robot dimensions -->
   <xacro:property name="PI" value="3.1415926535897931"/>
@@ -19,5 +23,5 @@
   <xacro:property name="axel_offset" value="0.05" />
     <xacro:property name="joint1_frame_rotation" value="0.0" />
-  <xacro:p_arm name="lio" parent="base_link" version="p_rob_2R">
+  <xacro:p_arm name="lio" parent="platform_base_link" version="p_rob_2R">
     <origin xyz="0 0 0.212" rpy="0 0 ${joint1_frame_rotation}" />
   </xacro:p_arm>

Commit message: put wheels in approximate positions

File: nsc_robot_description/urdf/nsc_robot_with_p_rob.xacro (robot description, xacro)
@@ -24,5 +24,5 @@
     <xacro:property name="joint1_frame_rotation" value="0.0" />
   <xacro:p_arm name="lio" parent="platform_base_link" version="p_rob_2R">
-    <origin xyz="0 0 0.212" rpy="0 0 ${joint1_frame_rotation}" />
+    <origin xyz="0 0 0.382" rpy="0 0 ${joint1_frame_rotation}" />
   </xacro:p_arm>
       <xacro:p_grip  name="lio"  parent="lio_gripper_interface_link" version="p_grip_2F" orientation="up"/>

File: nsc_robot_platform_description/urdf/platform_LIOc.urdf.xacro (robot description, xacro)
@@ -104,11 +104,11 @@
     <!-- A bunch of stuff cut -->
 </xacro:macro>
-<xacro:wheel parent_link="base_footprint" name_link="wheel_front_left" radius_wheel="${radius_wheel}" x="${depth/4}" y="${width/4}" z="${-height1/2 - radius_wheel}" rot_x="0" rot_y="1" rot_z="0" />
-<xacro:wheel parent_link="base_footprint" name_link="wheel_front_right" radius_wheel="${radius_wheel}" x="${depth/4}" y="${-width/4}" z="${-height1/2 - radius_wheel}" rot_x="0" rot_y="1" rot_z="0" />
+<xacro:wheel parent_link="platform_base_link" name_link="wheel_front_left" radius_wheel="${radius_wheel}" x="${depth/9}" y="${width/6}" z="${0.1 - radius_wheel}" rot_x="0" rot_y="1" rot_z="0" />
+<xacro:wheel parent_link="platform_base_link" name_link="wheel_front_right" radius_wheel="${radius_wheel}" x="${depth/9}" y="${-width/6}" z="${0.1 - radius_wheel}" rot_x="0" rot_y="1" rot_z="0" />
   <!-- wheel_back_right vertical joint-->
   <joint name="joint1_wheel_back_right" type="continuous">
-    <parent link="base_footprint"/>
+    <parent link="platform_base_link"/>
     <child link="wheel_back_right_bar"/>
-    <origin xyz="${-depth/4} ${-width/4} ${-height1/2}" rpy="0 0 0"/>
+    <origin xyz="${-depth/3} ${-width/8} 0.1" rpy="0 0 0"/>
     <axis xyz="0 0 1"/>
     <dynamics damping="0.7"/>
@@ -140,7 +140,7 @@
   <!-- wheel_back_left vertical joint-->
   <joint name="joint1_wheel_back_left" type="continuous">
-    <parent link="base_footprint"/>
+    <parent link="platform_base_link"/>
     <child link="wheel_back_left_bar"/>
-    <origin xyz="${-depth/4} ${width/4} ${-height1/2}" rpy="0 0 0"/>
+    <origin xyz="${-depth/3} ${width/8} 0.1" rpy="0 0 0"/>
     <axis xyz="0 0 1"/>
     <dynamics damping="0.7"/>

Commit message: added wheel controller - lio driving in home

File: nsc_robot_description/urdf/nsc_robot_with_p_rob.xacro (robot description, xacro)
@@ -87,3 +87,23 @@
     </actuator>
   </transmission>
+        <transmission name="trans7">
+    <type>transmission_interface/SimpleTransmission</type>
+    <joint name="base_to_wheel_front_left">
+      <hardwareInterface>EffortJointInterface</hardwareInterface>
+    </joint>
+    <actuator name="motor7">
+      <hardwareInterface>EffortJointInterface</hardwareInterface>
+      <mechanicalReduction>1</mechanicalReduction>
+    </actuator>
+  </transmission>
+            <transmission name="trans8">
+    <type>transmission_interface/SimpleTransmission</type>
+    <joint name="base_to_wheel_front_right">
+      <hardwareInterface>EffortJointInterface</hardwareInterface>
+    </joint>
+    <actuator name="motor8">
+      <hardwareInterface>EffortJointInterface</hardwareInterface>
+      <mechanicalReduction>1</mechanicalReduction>
+    </actuator>
+  </transmission>
 </robot>

Commit message: working 3d camera 2d screen

File: nsc_robot_description/urdf/nsc_robot_with_p_rob.xacro (robot description, xacro)
@@ -4,10 +4,5 @@
  <xacro:property name="robot_base_frame_rotation" value="$(env RDSCFG_fp_descriptions_robot_frame_rotation)"/>
  <xacro:property name="joint1_frame_rotation" value="$(env RDSCFG_fp_descriptions_j1_frame_rotation)"/>
- <xacro:include filename="$(find nsc_robot_p_arm_description)/urdf/p_arm.urdf.xacro" />
- <!-- <xacro:include filename="$(find nsc_robot_description)/urdf/nsc_robot_platform.xacro" /> -->
- <xacro:include filename="$(find nsc_robot_description)/urdf/nsc_robot_with_prob.gazebo" />
- <xacro:include filename="$(find nsc_robot_p_grip_description)/urdf/p_grip.urdf.xacro" />
- <xacro:include filename="$(find nsc_robot_platform_description)/urdf/platform_${robot_type}.urdf.xacro" />
- <!-- Constants for robot dimensions -->
+  <!-- Constants for robot dimensions -->
   <xacro:property name="PI" value="3.1415926535897931"/>
   <xacro:property name="mass" value="1" /> <!-- arbitrary value for mass -->
@@ -22,5 +17,14 @@
   <xacro:property name="camera_link" value="0.05" />
   <xacro:property name="axel_offset" value="0.05" />
-    <xacro:property name="joint1_frame_rotation" value="0.0" />
+  <xacro:property name="joint1_frame_rotation" value="0.0" />
+ <xacro:include filename="$(find nsc_robot_p_arm_description)/urdf/p_arm.urdf.xacro" />
+ <!-- <xacro:include filename="$(find nsc_robot_description)/urdf/nsc_robot_platform.xacro" /> -->
+ <xacro:include filename="$(find nsc_robot_description)/urdf/nsc_robot_with_prob.gazebo" />
+ <xacro:include filename="$(find nsc_robot_p_grip_description)/urdf/p_grip.urdf.xacro" />
+ <xacro:include filename="$(find nsc_robot_platform_description)/urdf/platform_${robot_type}.urdf.xacro" />
+ <xacro:include filename="$(find realsense2_description)/urdf/_d435.urdf.xacro" />
+ <sensor_d435 parent="platform_base_link">
+     <origin xyz="0.26 0.0 0.06" rpy="0 -0.3 0"/>
+ </sensor_d435>
   <xacro:p_arm name="lio" parent="platform_base_link" version="p_rob_2R">
     <origin xyz="0 0 0.382" rpy="0 0 ${joint1_frame_rotation}" />
@@ -107,3 +111,13 @@
     </actuator>
   </transmission>
+    <transmission name="trans9">
+    <type>transmission_interface/SimpleTransmission</type>
+    <joint name="lio_gripper_joint">
+      <hardwareInterface>EffortJointInterface</hardwareInterface>
+    </joint>
+    <actuator name="motor9">
+      <hardwareInterface>EffortJointInterface</hardwareInterface>
+      <mechanicalReduction>1</mechanicalReduction>
+    </actuator>
+  </transmission>
 </robot>
