Commit message: working inertia and coloured lio

File: nsc_robot_description/urdf/nsc_robot_platform.xacro (robot description, xacro)
@@ -17,7 +17,7 @@
     <inertial>
             <mass value="${mass}" />
-            <inertia ixx="1.0" ixy="0.0" ixz="0.0"
-                 iyy="1.0" iyz="0.0"
-                 izz="1.0" />
+            <inertia ixx="0.1" ixy="0.0" ixz="0.0"
+                 iyy="0.1" iyz="0.0"
+                 izz="0.1" />
     </inertial>
 </xacro:macro>

File: nsc_robot_description/urdf/nsc_robot_with_p_rob.xacro (robot description, xacro)
@@ -121,3 +121,13 @@
     </actuator>
   </transmission>
+        <transmission name="trans10">
+    <type>transmission_interface/SimpleTransmission</type>
+    <joint name="lio_passive_gripper_joint">
+      <hardwareInterface>EffortJointInterface</hardwareInterface>
+    </joint>
+    <actuator name="motor10">
+      <hardwareInterface>EffortJointInterface</hardwareInterface>
+      <mechanicalReduction>1</mechanicalReduction>
+    </actuator>
+  </transmission>
 </robot>

File: nsc_robot_p_arm_description/urdf/p_arm.urdf.xacro (robot description, xacro)
@@ -6,4 +6,5 @@
     name="p_arm"
     params="name parent version *origin">
+  <xacro:include filename="$(find nsc_robot_description)/urdf/materials.xacro" />
   <xacro:property
     name="config_path"
@@ -32,5 +33,5 @@
     <inertial>
       <origin
-        xyz="8.71294630254049E-05 0.277951295685675 -0.00113740271757783"
+        xyz="8.71294630254049E-05 0.0 -0.00113740271757783"
         rpy="0 0 0"/>
       <mass
@@ -49,5 +50,5 @@
           filename="package://nsc_robot_p_arm_description/meshes/${version}/link12.STL"/>
       </geometry>
-      <material name="blue"/>
+      <material name="orange_n"/>
     </visual>
     <collision>
@@ -88,5 +89,5 @@
           filename="package://nsc_robot_p_arm_description/meshes/${version}/link23.STL"/>
       </geometry>
-      <material name="white"/>
+      <material name="white_n"/>
     </visual>
     <collision>
@@ -112,5 +113,5 @@
     <inertial>
       <origin
-        xyz="8.71294630254052E-05 -0.313548704302934 -0.00113740271757783"
+        xyz="8.71294630254052E-05 0 -0.00113740271757783"
         rpy="0 0 0"/>
       <mass
@@ -129,5 +130,5 @@
           filename="package://nsc_robot_p_arm_description/meshes/${version}/link34.STL"/>
       </geometry>
-      <material name="blue"/>
+      <material name="orange_n"/>
     </visual>
     <collision>
@@ -153,5 +154,5 @@
     <inertial>
       <origin
-        xyz="8.71294630254052E-05 -0.313548704302934 -0.00113740271757783"
+        xyz="8.71294630254052E-05 0 -0.00113740271757783"
         rpy="0 0 0"/>
       <mass
@@ -170,5 +171,5 @@
           filename="package://nsc_robot_p_arm_description/meshes/${version}/link45.STL"/>
       </geometry>
-      <material name="white"/>
+      <material name="white_n"/>
     </visual>
     <collision>
@@ -193,5 +194,5 @@
   <link name="${name}_link56">
     <inertial>
-      <origin xyz="-8.71294630254049E-05 -0.588048704302934 0.00113740271757783"/>
+      <origin xyz="-8.71294630254049E-05 0 0.00113740271757783"/>
       <mass
         value="${parameters['link56_mass']}"/>
@@ -209,5 +210,5 @@
           filename="package://nsc_robot_p_arm_description/meshes/${version}/link56.STL"/>
       </geometry>
-      <material name="blue"/>
+      <material name="orange_n"/>
     </visual>
     <collision>
@@ -232,5 +233,5 @@
   <link name="${name}_link6G">
     <inertial>
-      <origin xyz="-0.00113740271757783 0.588048704302934 8.7129463025477E-05"/>
+      <origin xyz="-0.00113740271757783 0 8.7129463025477E-05"/>
       <mass
         value="${parameters['link6G_mass']}"/>
@@ -248,5 +249,5 @@
           filename="package://nsc_robot_p_arm_description/meshes/${version}/link6G.STL"/>
       </geometry>
-      <material name="white"/>
+      <material name="white_n"/>
     </visual>
     <collision>

File: nsc_robot_p_grip_description/urdf/p_grip.urdf.xacro (robot description, xacro)
@@ -169,7 +169,29 @@
     </link>
   </xacro:if>
+  <xacro:macro name="mimic_joint_plugin_gazebo" params="name_prefix parent_joint mimic_joint has_pid:=false multiplier:=1.0 offset:=0 sensitiveness:=0.0 max_effort:=1.0 robot_namespace:=''">
+    <gazebo>
+      <plugin name="${name_prefix}mimic_joint_plugin" filename="libroboticsgroup_gazebo_mimic_joint_plugin.so">
+        <joint>${parent_joint}</joint>
+        <mimicJoint>${mimic_joint}</mimicJoint>
+        <xacro:if value="${has_pid}">                     <!-- if set to true, PID parameters from "/gazebo_ros_control/pid_gains/${mimic_joint}" are loaded -->
+          <hasPID />
+        </xacro:if>
+        <multiplier>${multiplier}</multiplier>
+        <offset>${offset}</offset>
+        <sensitiveness>${sensitiveness}</sensitiveness>   <!-- if absolute difference between setpoint and process value is below this threshold, do nothing; 0.0 = disable [rad] -->
+        <maxEffort>${max_effort}</maxEffort>              <!-- only taken into account if has_pid:=true [Nm] -->
+        <xacro:unless value="${robot_namespace == ''}">
+          <robotNamespace>${robot_namespace}</robotNamespace>
+        </xacro:unless>
+      </plugin>
+    </gazebo>
+  </xacro:macro>
+  <!--
+  <xacro:mimic_joint_plugin_gazebo name_prefix="{name}_passive_gripper_joint"
+    parent_joint="${name}_gripper_joint" mimic_joint="{name}_passive_gripper_joint"
+    has_pid="true" multiplier="1.0" max_effort="10.0" /> robot_namespace="nsc_robot" -->
   <!-- The right finger simply mirrors the left one. -->
   <joint name="${name}_passive_gripper_joint" type="revolute">
-    <mimic joint="${name}_gripper_joint" multiplier="-1" offset="0"/>
+    <!-- <mimic joint="${name}_gripper_joint" multiplier="-1" offset="0"/> -->
     <origin
             xyz="${parameters['right_finger_translation']}"
@@ -177,5 +199,10 @@
     <parent link="${name}_gripper_link"/>
     <child link="${name}_right_finger"/>
-    <limit effort="1000.0" lower="0" upper="0.52" velocity="170"/>
+    <!-- <limit effort="1000.0" lower="0" upper="0.52" velocity="170"/> -->
+    <limit
+      effort="${parameters['effort_limit']}"
+      lower="${parameters['lower_angle_limit'] * pi/180}"
+      upper="${parameters['upper_angle_limit'] * -pi/180}"
+      velocity="${parameters['velocity_limit'] * pi/180}"/>
     <axis xyz="0 0 1"/>
   </joint>

File: nsc_robot_platform_description/urdf/platform_LIOc.urdf.xacro (robot description, xacro)
@@ -74,7 +74,7 @@
     <inertial>
             <mass value="${mass}" />
-            <inertia ixx="1.0" ixy="0.0" ixz="0.0"
-                 iyy="1.0" iyz="0.0"
-                 izz="1.0" />
+            <inertia ixx="0.2" ixy="0.0" ixz="0.0"
+                 iyy="0.2" iyz="0.0"
+                 izz="0.2" />
     </inertial>
 </xacro:macro>

Commit message: optimized mobile_platform inertias of wheels

File: nsc_robot_description/urdf/nsc_robot_platform.xacro (robot description, xacro)
@@ -1,7 +1,10 @@
 <?xml version="1.0"?>
 <robot name="nsc_robot" xmlns:xacro="http://www.ros.org/wiki/xacro">
+ <xacro:include filename="$(find onebot_description)/urdf/caster.urdf.xacro" />
  <!-- Constants for robot dimensions -->
   <xacro:property name="PI" value="3.1415926535897931"/>
-  <xacro:property name="mass" value="1" /> <!-- arbitrary value for mass -->
+  <xacro:property name="mass" value="0.1" /> <!-- arbitrary value for mass -->
+  <xacro:property name="mass_wheel" value="0.2" /> <!-- arbitrary value for mass -->
+  <xacro:property name="mass_base" value="30" />
   <xacro:property name="width" value="0.8" />
   <xacro:property name="depth" value="1.0" />
@@ -14,13 +17,22 @@
   <xacro:property name="camera_link" value="0.05" />
   <xacro:property name="axel_offset" value="0.05" />
-<xacro:macro name="default_inertial" params="mass">
+  <xacro:arg name="mesh_enabled" default="false" />
+<xacro:macro name="default_inertial_wheel" params="mass radius_wheel length_wheel" >
+    <inertial>
+            <mass value="${mass}" />
+            <inertia ixx="${0.25 * mass * radius_wheel**2 + 1/12 * mass * length_wheel**2}" ixy="0.0" ixz="0.0"
+                 iyy="${1/2 * mass * radius_wheel**2}" iyz="0.0"
+                 izz="${0.25 * mass * radius_wheel**2 + 1/12 * mass * length_wheel**2}" />
+    </inertial>
+</xacro:macro>
+<xacro:macro name="default_inertial" params="mass" >
     <inertial>
             <mass value="${mass}" />
             <inertia ixx="0.1" ixy="0.0" ixz="0.0"
-                 iyy="0.1" iyz="0.0"
+                 iyy="0.1"
                  izz="0.1" />
     </inertial>
 </xacro:macro>
-<xacro:macro name="wheel" params="parent_link name_link radius_wheel x y z rot_x rot_y rot_z">
+<xacro:macro name="wheel" params="parent_link name_link radius_wheel mass_wheel length_wheel x y z rot_x rot_y rot_z">
     <link name="${name_link}_leg">
         <visual>
@@ -37,5 +49,5 @@
             <origin xyz="0 0 0" rpy="${PI/2} 0 0"/>
         </collision>
-        <xacro:default_inertial mass="1"/>
+        <xacro:default_inertial_wheel mass="${mass_wheel}" radius_wheel="${radius_wheel}" length_wheel="${length_wheel}"/>
     </link>
     <joint name="base_to_${name_link}" type="continuous">
@@ -47,6 +59,6 @@
     <!-- A bunch of stuff cut -->
 </xacro:macro>
-<xacro:wheel parent_link="base_link" name_link="wheel_front_left" radius_wheel="${radius_wheel}" x="${depth/4}" y="${width/4}" z="${-height1/2 - radius_wheel}" rot_x="0" rot_y="1" rot_z="0" />
-<xacro:wheel parent_link="base_link" name_link="wheel_front_right" radius_wheel="${radius_wheel}" x="${depth/4}" y="${-width/4}" z="${-height1/2 - radius_wheel}" rot_x="0" rot_y="1" rot_z="0" />
+<xacro:wheel parent_link="base_link" name_link="wheel_front_left" radius_wheel="${radius_wheel}" mass_wheel="${mass_wheel}" length_wheel="${length_wheel}" x="${depth/4}" y="${width/4}" z="${-height1/2 - radius_wheel}" rot_x="0" rot_y="1" rot_z="0" />
+<xacro:wheel parent_link="base_link" name_link="wheel_front_right" radius_wheel="${radius_wheel}" mass_wheel="${mass_wheel}" length_wheel="${length_wheel}" x="${depth/4}" y="${-width/4}" z="${-height1/2 - radius_wheel}" rot_x="0" rot_y="1" rot_z="0" />
   <!-- Base Link -->
   <link name="base_link">
@@ -66,5 +78,5 @@
     <inertial>
       <origin xyz="0 0 0" rpy="0 0 0"/>
-      <mass value="${mass}"/>
+      <mass value="${mass_base}"/>
       <inertia
           ixx="${mass / 12.0 * (width*width + height1*height1)}" ixy="0.0" ixz="0.0"
@@ -73,5 +85,11 @@
     </inertial>
   </link>
-  <!-- wheel_back_right vertical joint-->
+    <xacro:caster caster_prefix="left_rear" parent_link="base_link" >
+        <origin xyz="${-depth/4} ${width/4} ${-height1/2 - 2 * radius_wheel + 0.065}" rpy="0 0 0" />
+    </xacro:caster>
+    <xacro:caster caster_prefix="right_rear" parent_link="base_link" >
+        <origin xyz="${-depth/4} ${-width/4} ${-height1/2 - 2 * radius_wheel + 0.065}" rpy="0 0 0" />
+    </xacro:caster>
+  <!-- wheel_back_right vertical joint
   <joint name="joint1_wheel_back_right" type="continuous">
     <parent link="base_link"/>
@@ -105,5 +123,6 @@
   </link>
 <xacro:wheel parent_link="wheel_back_right_bar" name_link="wheel_back_right" radius_wheel="${radius_wheel}" x="0" y="0" z="${-height2}" rot_x="0" rot_y="1" rot_z="0" />
-  <!-- wheel_back_left vertical joint-->
+  -->
+  <!-- wheel_back_left vertical joint
   <joint name="joint1_wheel_back_left" type="continuous">
     <parent link="base_link"/>
@@ -137,3 +156,4 @@
   </link>
 <xacro:wheel parent_link="wheel_back_left_bar" name_link="wheel_back_left" radius_wheel="${radius_wheel}" x="0" y="0" z="${-height2}" rot_x="0" rot_y="1" rot_z="0" />
+  -->
 </robot>

File: nsc_robot_description/urdf/nsc_robot_with_p_rob.xacro (robot description, xacro)
@@ -23,8 +23,10 @@
  <xacro:include filename="$(find nsc_robot_p_grip_description)/urdf/p_grip.urdf.xacro" />
  <xacro:include filename="$(find nsc_robot_platform_description)/urdf/platform_${robot_type}.urdf.xacro" />
+ <!--
  <xacro:include filename="$(find realsense2_description)/urdf/_d435.urdf.xacro" />
  <sensor_d435 parent="platform_base_link">
      <origin xyz="0.26 0.0 0.06" rpy="0 -0.3 0"/>
  </sensor_d435>
+  -->
   <xacro:p_arm name="lio" parent="platform_base_link" version="p_rob_2R">
     <origin xyz="0 0 0.382" rpy="0 0 ${joint1_frame_rotation}" />

Commit message: first working prototype of Q_learning control without learning

File: nsc_robot_description/urdf/nsc_robot_platform.xacro (robot description, xacro)
@@ -2,4 +2,5 @@
 <robot name="nsc_robot" xmlns:xacro="http://www.ros.org/wiki/xacro">
  <xacro:include filename="$(find onebot_description)/urdf/caster.urdf.xacro" />
+ <xacro:include filename="$(find nsc_robot_description)/urdf/nsc_robot_platform.gazebo" />
  <!-- Constants for robot dimensions -->
   <xacro:property name="PI" value="3.1415926535897931"/>
@@ -157,3 +158,23 @@
 <xacro:wheel parent_link="wheel_back_left_bar" name_link="wheel_back_left" radius_wheel="${radius_wheel}" x="0" y="0" z="${-height2}" rot_x="0" rot_y="1" rot_z="0" />
   -->
+  <transmission name="tran1">
+    <type>transmission_interface/SimpleTransmission</type>
+    <joint name="base_to_wheel_front_left">
+      <hardwareInterface>EffortJointInterface</hardwareInterface>
+    </joint>
+    <actuator name="motor1">
+      <hardwareInterface>EffortJointInterface</hardwareInterface>
+      <mechanicalReduction>1</mechanicalReduction>
+    </actuator>
+  </transmission>
+    <transmission name="tran2">
+    <type>transmission_interface/SimpleTransmission</type>
+    <joint name="base_to_wheel_front_right">
+      <hardwareInterface>EffortJointInterface</hardwareInterface>
+    </joint>
+    <actuator name="motor2">
+      <hardwareInterface>EffortJointInterface</hardwareInterface>
+      <mechanicalReduction>1</mechanicalReduction>
+    </actuator>
+  </transmission>
 </robot>
